File: hardware/kicad/connectors.kicad_sch (KiCad schematic)
At the start: 9 parts, among them J701 RC receiver, J702 GPS, J703 Aux I2C, J704 Buzzer, J705 LED strip, Q701 2N7002

Commit message: Verify IMU footprint; fix Block 7 LED and buzzer parts
- U301 ICM-42688-P footprint verified against DS-000347 Rev 1.2 (LGA-14
  2.5x3.0, 0.5 mm pitch, C-C 2.525/2.025) — Bosch LGA-14 is a correct mate
- D702 S2M 2A silicon in series on J705 strip VDD: drops strip to ~4.3 V so
  WS2812 VIH is reachable from the 3V3 data line
- Q701 2N7002 -> AO3400A for buzzer current headroom
- J705 note records the real limit: ~1 A / ~16 LEDs, capped by the JST-SH

Co-Authored-By: Claude Sonnet 5 <noreply@anthropic.com>
Claude-Session: https://claude.ai/code/session_0171uwNh8K8uwZuWio9f35u1
Parts:
- added D702: S2M, Diode_SMD:D_SMA, symbol Device:D
- Q701: value 2N7002 -> AO3400A; symbol Transistor_FET:2N7002 -> Transistor_FET:AO3400A; LCSC C8545 -> C20917; MPN 2N7002 -> AO3400A; Manufacturer Jiangsu Changjing Electronics -> Alpha & Omega Semiconductor
Connections:
- net +5V: now also D702.2 (A); no longer J705.1 (Pin_1)
- new net: D702.1 (K), J705.1 (Pin_1)
Other:
- note added: "Buzzer low-side switch: Q701 AO3400A (SOT-23, 30 V, 5.7 A, ~28 mOhm) - headroom for louder / higher-current buzzers vs the old 2N7002. Gate from BUZZER (PB8) with R701 10k pull-down. D701 1N4148W flyback across the buzzer, cathode to +5V. J704: 1=+5V 2=buzzer- (BUZZ_N)."
- note added: "J705 LED strip - WS2812. D702 (S2M, 2 A silicon rectifier, SMA) in series on strip VDD: 5 V - ~0.7 V @ 0.5 A -> strip runs at ~4.3 V, so WS2812 VIH (~0.7*VDD ~= 3.0 V) is within reach of the 3V3 LED_DATA line (PA8 via R702 330R). A Schottky (~0.3 V) would give ~4.7 V and leave VIH marginal - silicon is required. Real current limit: the JST-SH connector (SM03B-SRSS-TB, 1 A / contact) caps strip dr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"
- note removed: "Buzzer low-side switch: Q701 2N7002, gate from BUZZER (PB8) with R701 10k pull-down. D701 1N4148W flyback across the buzzer, cathode to +5V. J704: 1=+5V 2=buzzer- (BUZZ_N)."
- note removed: "J705 LED strip — WS2812; 5 V strip driven from a 3.3 V pin (PA8), level shift may be needed for long runs. R702 330R series on data. 1=+5V 2=GND 3=DATA (LED_STRIP via R702)."
Changed lines of the file:
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@@
 	(paper "A4")
-	(junction
-		(at 165.1 177.8)
-		(diameter 0)
-		(color 0 0 0 0)
-	)
 	(junction
 		(at 165.1 180.34)
@@
 	(wire
 		(pts
-			(xy 165.1 177.8)
-			(xy 162.56 177.8)
-		)
-	)
-	(wire
-		(pts
 			(xy 165.1 180.34)
 			(xy 162.56 180.34)
@@
 		)
 	)
+	(wire
+		(pts
+			(xy 151.13 177.8)
+			(xy 148.59 177.8)
+		)
+	)
+	(text "J701 RC receiver — CRSF/ELRS external receiver, UART3 (USART3 PB10/PB11).\n1=+5V  2=GND  3=RX_UART_TX  4=RX_UART_RX."
+		(at 120 30 0)
+		(effects
+			(font
+				(size 1.27 1.27)
+			)
+			(justify left bottom)
+		)
+	)
+	(text "J702 GPS — USART2, PA2 (USART2_TX -> GPS_TX) / PA3 (USART2_RX -> GPS_RX).\nFree UART pair per pinmap (\"PA2/PA3 spare UART2\"). 1=+5V 2=GND 3=GPS_TX 4=GPS_RX."
+		(at 120 75 0)
+		(effects
+			(font
+				(size 1.27 1.27)
+			)
+			(justify left bottom)
+		)
+	)
+	(text "J703 aux I2C — shares I2C1 with U401; pull-ups already on the baro sheet, do not add more.\n1=+5V  2=GND  3=I2C1_SCL  4=I2C1_SDA."
+		(at 120 120 0)
+		(effects
+			(font
+				(size 1.27 1.27)
+			)
+			(justify left bottom)
+		)
+	)
 	(label "BUZZ_N"
 		(at 77.47 97.79 0)
@@
 		)
 	)
+	(global_label "GND"
+		(shape input)
+		(at 162.56 180.34 180)
+		(effects
+			(font
+				(size 1.27 1.27)
+			)
+			(justify right)
+		)
+	)
+	(global_label "BUZZER"
+		(shape input)
+		(at 67.31 105.41 180)
+		(effects
+			(font
+				(size 1.27 1.27)
+			)
+			(justify right)
+		)
+	)
+	(global_label "GND"
+		(shape input)
+		(at 77.47 113.03 0)
+		(effects
+			(font
+				(size 1.27 1.27)
+			)
+			(justify left)
+		)
+	)
+	(global_label "GND"
+		(shape input)
+		(at 59.69 125.73 0)
+		(effects
+			(font
+				(size 1.27 1.27)
+			)
+			(justify left)
+		)
+	)
 	(global_label "+5V"
 		(shape input)
-		(at 162.56 177.8 180)
-		(effects
-			(font
-				(size 1.27 1.27)
-			)
-			(justify right)
-		)
-	)
-	(global_label "GND"
-		(shape input)
-		(at 162.56 180.34 180)
-		(effects
-			(font
-				(size 1.27 1.27)
-			)
-			(justify right)
-		)
-	)
-	(global_label "BUZZER"
-		(shape input)
-		(at 67.31 105.41 180)
-		(effects
-			(font
-				(size 1.27 1.27)
-			)
-			(justify right)
-		)
-	)
-	(global_label "GND"
-		(shape input)
-		(at 77.47 113.03 0)
+		(at 102.87 95.25 180)
+		(effects
+			(font
+				(size 1.27 1.27)
+			)
+			(justify right)
+		)
+	)
+	(global_label "+5V"
+		(shape input)
+		(at 95.25 86.36 0)
 		(effects
 			(font
@@
 		)
 	)
-	(global_label "GND"
-		(shape input)
-		(at 59.69 125.73 0)
-		(effects
-			(font
-				(size 1.27 1.27)
-			)
-			(justify left)
+	(global_label "LED_STRIP"
+		(shape input)
+		(at 133.35 175.26 180)
+		(effects
+			(font
+				(size 1.27 1.27)
+			)
+			(justify right)
 		)
 	)
 	(global_label "+5V"
 		(shape input)
-		(at 102.87 95.25 180)
-		(effects
-			(font
-				(size 1.27 1.27)
-			)
-			(justify right)
-		)
-	)
-	(global_label "+5V"
-		(shape input)
-		(at 95.25 86.36 0)
-		(effects
-			(font
-				(size 1.27 1.27)
-			)
-			(justify left)
-		)
-	)
-	(global_label "LED_STRIP"
-		(shape input)
-		(at 133.35 175.26 180)
-		(effects
-			(font
-				(size 1.27 1.27)
-			)
-			(justify right)
-		)
-	)
-  (text "J701 RC receiver — CRSF/ELRS external receiver, UART3 (USART3 PB10/PB11).\n1=+5V  2=GND  3=RX_UART_TX  4=RX_UART_RX."
-    (at 120 30 0)
+		(at 148.59 177.8 180)
+		(effects
+			(font
+				(size 1.27 1.27)
+			)
+			(justify right)
+		)
+	)
+(wire
+		(pts
+			(xy 158.75 177.8) (xy 165.1 177.8)
+		)
+		(stroke
+			(width 0)
+			(type default)
+		)
+	)
+  (text "Buzzer low-side switch: Q701 AO3400A (SOT-23, 30 V, 5.7 A, ~28 mOhm) - headroom\nfor louder / higher-current buzzers vs the old 2N7002.  Gate from BUZZER (PB8)\nwith R701 10k pull-down.  D701 1N4148W flyback across the buzzer, cathode to +5V.\nJ704: 1=+5V  2=buzzer- (BUZZ_N)."
+    (at 45 62 0)
     (effects (font (size 1.27 1.27)) (justify left bottom))
   )
-  (text "J702 GPS — USART2, PA2 (USART2_TX -> GPS_TX) / PA3 (USART2_RX -> GPS_RX).\nFree UART pair per pinmap (\"PA2/PA3 spare UART2\"). 1=+5V 2=GND 3=GPS_TX 4=GPS_RX."
-    (at 120 75 0)
-    (effects (font (size 1.27 1.27)) (justify left bottom))
-  )
-  (text "J703 aux I2C — shares I2C1 with U401; pull-ups already on the baro sheet, do not add more.\n1=+5V  2=GND  3=I2C1_SCL  4=I2C1_SDA."
-    (at 120 120 0)
-    (effects (font (size 1.27 1.27)) (justify left bottom))
-  )
-  (text "J705 LED strip — WS2812; 5 V strip driven from a 3.3 V pin (PA8),\nlevel shift may be needed for long runs. R702 330R series on data.\n1=+5V  2=GND  3=DATA (LED_STRIP via R702)."
-    (at 120 163 0)
-    (effects (font (size 1.27 1.27)) (justify left bottom))
-  )
-  (text "Buzzer low-side switch: Q701 2N7002, gate from BUZZER (PB8) with R701 10k\npull-down. D701 1N4148W flyback across the buzzer, cathode to +5V.\nJ704: 1=+5V  2=buzzer- (BUZZ_N)."
-    (at 45 62 0)
+  (text "J705 LED strip - WS2812.  D702 (S2M, 2 A silicon rectifier, SMA) in series on\nstrip VDD: 5 V - ~0.7 V @ 0.5 A -> strip runs at ~4.3 V, so WS2812 VIH\n(~0.7*VDD ~= 3.0 V) is within reach of the 3V3 LED_DATA line (PA8 via R702 330R).\nA Schottky (~0.3 V) would give ~4.7 V and leave VIH marginal - silicon is required.\nReal current limit: the JST-SH connector (SM03B-SRSS-TB, 1 A / contact) caps strip\ndraw at ~1 A = roughly 16 WS2812 at full white (~60 mA each).  D702 must be rated\nabove that - S2M (2 A) clears it.  Feed a longer strip from its own 5 V, not J705.\n1=+5V (via D702)  2=GND  3=DATA (LED_STRIP via R702)."
+    (at 115 160 0)
     (effects (font (size 1.27 1.27)) (justify left bottom))
   )
@@
 	)
 	(symbol
-		(lib_id "Transistor_FET:2N7002")
+		(lib_id "Transistor_FET:AO3400A")
 		(at 74.93 105.41 0)
 		(unit 1)
@@
 			)
 		)
-		(property "Value" "2N7002"
+		(property "Value" "AO3400A"
 			(at 80.01 105.41 0)
 			(effects
@@
 			)
 		)
-		(property "LCSC" "C8545"
+		(property "LCSC" "C20917"
 			(at 74.93 105.41 0)
 			(hide yes)
@@
 			)
 		)
-		(property "MPN" "2N7002"
+		(property "MPN" "AO3400A"
 			(at 74.93 105.41 0)
 			(hide yes)
@@
 			)
 		)
-		(property "Manufacturer" "Jiangsu Changjing Electronics"
+		(property "Manufacturer" "Alpha & Omega Semiconductor"
 			(at 74.93 105.41 0)
 			(hide yes)
@@
 		)
 	)
+	(symbol
+		(lib_id "Device:D")
+		(at 154.94 177.8 180)
+		(unit 1)
+		(in_bom yes)
+		(on_board yes)
+		(dnp no)
+		(property "Reference" "D702"
+			(at 154.94 180.34 0)
+			(effects
+				(font
+					(size 1.27 1.27)
+				)
+			)
+		)
+		(property "Value" "S2M"
+			(at 154.94 175.26 0)
+			(effects
+				(font
+					(size 1.27 1.27)
+				)
+			)
+		)
+		(property "Footprint" "Diode_SMD:D_SMA"
+			(at 154.94 177.8 0)
+			(hide yes)
+			(effects
+				(font
+					(size 1.27 1.27)
+				)
+			)
+		)
+		(property "Datasheet" ""
+			(at 154.94 177.8 0)
+			(hide yes)
+			(effects
+				(font
+					(size 1.27 1.27)
+				)
+			)
+		)
+		(property "Description" "Diode"
+			(at 154.94 177.8 0)
+			(hide yes)
+			(effects
+				(font
+					(size 1.27 1.27)
+				)
+			)
+		)
+		(instances
+			(project "connectors"
+				(path "20e6064d-7924-44bd-8a09-738759519a1e"
+					(reference "D702")
+					(unit 1)
+				)
+			)
+		)
+		(property "LCSC" "C18905"
+			(at 154.94 177.8 0)
+			(hide yes)
+			(effects
+				(font
+					(size 1.27 1.27)
+				)
+			)
+		)
+		(property "MPN" "S2M"
+			(at 154.94 177.8 0)
+			(hide yes)
+			(effects
+				(font
+					(size 1.27 1.27)
+				)
+			)
+		)
+		(property "Manufacturer" "MDD(Microdiode Semiconductor)"
+			(at 154.94 177.8 0)
+			(hide yes)
+			(effects
+				(font
+					(size 1.27 1.27)
+				)
+			)
+		))
 )
