File: hardware/kicad/dronekit-pro.kicad_sch (KiCad schematic)
At the start: 31 parts, among them J101 3S–4S LiPo (11.1–16.8 V), Q101 AOD4185, U101 MP2307DN-LF-Z, U102 RT9013-33GB, U103 AP7361C-33E, U803 LM66100DCKR

Commit message: Design review fixes: EN divider, +5V OR sizing, +5V bulk
- R106 43k -> 39k: MP2307 EN lockout 2.5V typ gives ~8.9 V turn-on and
  keeps EN < 6 V abs-max to 20 V input (was 6.0 V, zero margin)
- U803 LM66100 -> LM74700 + Q803 AO3400A: 1.5 A ceiling was below the
  ~1.9 A worst-case +5V budget; now FET-limited ~5 A at ~53 mV
- C113 22uF on the +5V OR node (was ~2 uF of LDO input caps only)
- ERC power_output x power_output reverted to Error; +5V now has a
  single power-output pin

Co-Authored-By: Claude Sonnet 5 <noreply@anthropic.com>
Claude-Session: https://claude.ai/code/session_0171uwNh8K8uwZuWio9f35u1
Parts:
- removed U803: LM66100DCKR, Package_TO_SOT_SMD:SOT-363_SC-70-6, symbol Power_Management:LM66100DCK
- added C113: 22uF, Capacitor_SMD:C_0805_2012Metric, symbol Device:C
- added C803, C804: 100nF, Capacitor_SMD:C_0603_1608Metric, symbol Device:C
- added Q803: AO3400A, Package_TO_SOT_SMD:SOT-23, symbol Transistor_FET:AO3400A
- added U803: LM74700QDBVRQ1, Package_TO_SOT_SMD:SOT-23-6, symbol Power_Management:LM74700
- R105: LCSC (none) -> C25803; MPN (none) -> 0603WAF1003T5E; Manufacturer (none) -> UNI-ROYAL
- R106: value 43k -> 39k; LCSC (none) -> C23153; MPN (none) -> 0603WAF3902T5E; Manufacturer (none) -> UNI-ROYAL
Connections:
- net +5V: now also C113.1, C804.1, Q803.3 (D), U803.4 (CATHODE)
- net +5V_BUCK: now also C803.2, C804.2, Q803.2 (S), U803.3 (EN), U803.6 (ANODE)
- net GND: now also C113.2, U803.2 (GND)
- new net U803_GATE: Q803.1 (G), U803.5 (GATE)
- new net U803_VCAP: C803.1, U803.1 (VCAP)
- no-connect marks 4 -> 2
Other:
- note added: "Buck-side OR-ing ideal diode (U803 LM74700-Q1 + Q803 AO3400A). Per LM74700-Q1 datasheet (SNOSD17G) Table 5-1 / Fig 5-1 / Fig 10-18: ANODE (pin 6) = input, connect to FET SOURCE -> +5V_BUCK (Q803.S) CATHODE (pin 4) = output, connect to FET DRAIN -> +5V (Q803.D) EN (pin 3) -> ANODE (always on). GATE (pin 5) -> Q803.G. C803 100nF charge-pump cap between VCAP and ANODE (datasheet 9.3.2). C804 100nF A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"
- note added: "Input 3S-4S LiPo (11.1-16.8 V). R105 100k / R106 39k on the MP2307 EN pin: EN_BUCK = VBAT_SW x 39/139 = x0.281. This is a REGULATOR BROWNOUT / EN-lockout threshold, NOT LiPo cell protection - there is no per-cell monitoring. MP2307 (r1.9): EN LOCKOUT (buck starts/stops switching) = 2.5 V typ, 2.2 / 2.7 V min/max; EN SHUTDOWN = 1.5 V typ. Buck stops switching when VBAT_SW falls to ~8.9 V typ, with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"
- note removed: "Buck-side OR-ing ideal diode (U803, LM66100DCKR): MP2307 output = +5V_BUCK (L101 / C105 / C106). FB (R102/R103) senses +5V_BUCK, so the buck regulates ITS OWN output to 5.0 V (no cross-coupling to the USB source). U803: VIN=+5V_BUCK, VOUT=+5V, CE tied to VOUT, GND to GND -> reverse-current-blocking ideal diode, ~48 mV drop at 0.5 A. Why: MP2307 is synchronous; its integrated high-side FET body di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"
- note removed: "Input 3S–4S (11.1–16.8 V). R105/R106 divider sets EN UVLO ≈ 9 V; EN < 6 V at 16.8 V."
