File: hardware/kicad/dronekit-pro.kicad_sch (KiCad schematic)
At the start: 35 parts, among them J101 3S–4S LiPo (11.1–16.8 V), Q101 AOD4185, Q803 AO3400A, U101 MP2307DN-LF-Z, U102 RT9013-33GB, U103 AP7361C-33E, U803 LM74700QDBVRQ1

Commit message: Review fixes: series protection R, I2C1 2.2k, C102 50V, gate & buck soft-start
7.f - PA2/PA3 = TTa (not 5V tolerant), PD2 = FT (5V tolerant) per STM32F405
DS8626. Add series R on the STM32 pin side: R205 1k ESC_TLM, R206 1k GPS_TX,
R207 1k GPS_RX (limits fault injection into PA2/PA3 to ~1.2 mA on a 5V UART).

3.a - Cross-domain series R: R208 470 BRIDGE_TX, R209 470 BRIDGE_RX, R210 470
ESP_STM_NRST (R203 pull-down + Q201 gate kept on the local node -> ESP-absent
fail-safe preserved).

6.a - I2C1 pull-ups R401/R402 4.7k -> 2.2k (C4190). With J703 cabled
(~90-100 pF): t_r ~= 186 ns < 300 ns (400 kHz); sink 1.4 mA at VOL.

1.a - C102 10uF 25V -> 50V (C138687), for 4S input transients + DC-bias
derating.

7.a - Inrush handled by a BUILD REQUIREMENT: anti-spark XT60/XT90 on the
battery lead (a single reverse-polarity P-FET cannot soft-start plug-in
inrush - body diode is forward). C114 100nF gate-source stays for a
controlled ~7 ms gate turn-on / softer VBAT_SW rise. J101 annotated.

MP2307 SS: C115 100nF on the SS pin (was left open). t_ss ~= 15 ms per r1.9
-> +5V ramps 0->5 V charging C105+C113 (~46 uF) at ~15 mA, not the ~4 A
current limit. Project symbol MP2307DN pin 8 corrected NC -> SS (passive).

ERC: 0 errors / 0 isolated_pin_label / 2 known pin_to_pin warnings.

Co-Authored-By: Claude Sonnet 5 <noreply@anthropic.com>
Claude-Session: https://claude.ai/code/session_0171uwNh8K8uwZuWio9f35u1
Parts:
- added C114, C115: 100nF, Capacitor_SMD:C_0603_1608Metric, symbol Device:C
- C102: value 10uF/25V -> 10uF/50V; LCSC (none) -> C138687; MPN (none) -> CL32B106KBJNNNE; Manufacturer (none) -> Samsung Electro-Mechanics; Voltage (none) -> 50V
- J101: Note (none) -> Battery lead MUST use an anti-spark XT60/XT90 connector - n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
Connections:
- net GND: now also C115.2
- net QGATE: now also C114.1
- net VBAT_SW: now also C114.2
- net SS_BUCK: now reaches U101.8 (SS)
- net SS_BUCK: now also C115.1
- no-connect marks 2 -> 1
Other:
- note added: "INRUSH / SOFT-START (7.a decision): BUILD REQUIREMENT: the battery lead MUST use an anti-spark XT60/XT90 connector (pre-charge resistor in the plug). Plug-in inrush is NOT limited on-board: Q101's body diode (VBAT->VBAT_SW, forward) charges C101 100uF + C102 10uF + C103 through the diode regardless of the gate (I_peak ~ 170-340 A for ~5-30 us, spark ~15 mJ at 16.8 V). A single reverse-polarity P-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"
