File: hardware/kicad/baro_flash.kicad_sch (KiCad schematic)
At the start: 10 parts, among them U401 DPS368XTSA1, U402 W25Q128JVSIQ

Commit message: Review fixes: series protection R, I2C1 2.2k, C102 50V, gate & buck soft-start
7.f - PA2/PA3 = TTa (not 5V tolerant), PD2 = FT (5V tolerant) per STM32F405
DS8626. Add series R on the STM32 pin side: R205 1k ESC_TLM, R206 1k GPS_TX,
R207 1k GPS_RX (limits fault injection into PA2/PA3 to ~1.2 mA on a 5V UART).

3.a - Cross-domain series R: R208 470 BRIDGE_TX, R209 470 BRIDGE_RX, R210 470
ESP_STM_NRST (R203 pull-down + Q201 gate kept on the local node -> ESP-absent
fail-safe preserved).

6.a - I2C1 pull-ups R401/R402 4.7k -> 2.2k (C4190). With J703 cabled
(~90-100 pF): t_r ~= 186 ns < 300 ns (400 kHz); sink 1.4 mA at VOL.

1.a - C102 10uF 25V -> 50V (C138687), for 4S input transients + DC-bias
derating.

7.a - Inrush handled by a BUILD REQUIREMENT: anti-spark XT60/XT90 on the
battery lead (a single reverse-polarity P-FET cannot soft-start plug-in
inrush - body diode is forward). C114 100nF gate-source stays for a
controlled ~7 ms gate turn-on / softer VBAT_SW rise. J101 annotated.

MP2307 SS: C115 100nF on the SS pin (was left open). t_ss ~= 15 ms per r1.9
-> +5V ramps 0->5 V charging C105+C113 (~46 uF) at ~15 mA, not the ~4 A
current limit. Project symbol MP2307DN pin 8 corrected NC -> SS (passive).

ERC: 0 errors / 0 isolated_pin_label / 2 known pin_to_pin warnings.

Co-Authored-By: Claude Sonnet 5 <noreply@anthropic.com>
Claude-Session: https://claude.ai/code/session_0171uwNh8K8uwZuWio9f35u1
Parts:
- R401, R402: value 4.7k -> 2.2k; LCSC C23162 -> C4190; MPN 0603WAF4701T5E -> 0603WAF2201T5E
Other:
- note added: "I2C1 pull-ups: R401 (SCL) / R402 (SDA) = 2.2k to +3V3_SYS, the ONLY pull-ups on I2C1. Master = STM32 PB6/PB7. 2.2k chosen for the J703 aux-I2C header: with a cabled external device (on-board ~30 pF + J703 cable/device ~35-65 pF ~= 90-100 pF worst case) t_r = 0.847*2.2k*100pF ~= 186 ns, under the 400 kHz fast-mode limit of 300 ns. Sink current at VOL: (3.3 - 0.2)/2.2k ~= 1.4 mA per line, well with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"
- note removed: "I2C1 pull-ups: R401 (SCL) and R402 (SDA), 4.7k to +3V3_SYS, are the ONLY pull-ups on I2C1. Bus master = STM32 PB6/PB7 (STM32 Core sheet). U401: DPS368 drawn with the BMP280 symbol (pin-identical per DPS368 DS v1.1 Table 2). VERIFY LGA-8 land pattern vs DPS368 DS Fig.18 before layout."
Changed lines of the file:
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@@
 		)
 	)
-  (text "I2C1 pull-ups: R401 (SCL) and R402 (SDA), 4.7k to +3V3_SYS, are the\nONLY pull-ups on I2C1. Bus master = STM32 PB6/PB7 (STM32 Core sheet).\nU401: DPS368 drawn with the BMP280 symbol (pin-identical per DPS368 DS\nv1.1 Table 2). VERIFY LGA-8 land pattern vs DPS368 DS Fig.18 before layout."
-    (at 105.41 125.73 0)
+  (text "SPI3 dedicated to blackbox flash; FLASH_CS = PA15."
+    (at 168.91 185.42 0)
     (effects (font (size 1.27 1.27)) (justify left bottom))
   )
-  (text "SPI3 dedicated to blackbox flash; FLASH_CS = PA15."
-    (at 168.91 185.42 0)
+  (text "I2C1 pull-ups: R401 (SCL) / R402 (SDA) = 2.2k to +3V3_SYS, the ONLY pull-ups\non I2C1.  Master = STM32 PB6/PB7.  2.2k chosen for the J703 aux-I2C header:\nwith a cabled external device (on-board ~30 pF + J703 cable/device ~35-65 pF\n~= 90-100 pF worst case) t_r = 0.847*2.2k*100pF ~= 186 ns, under the 400 kHz\nfast-mode limit of 300 ns.  Sink current at VOL: (3.3 - 0.2)/2.2k ~= 1.4 mA\nper line, well within the I2C >=3 mA sink of the STM32 and the DPS368.\nU401 = DPS368 drawn with the BMP280 symbol (pin-identical per DPS368 DS v1.1\nTable 2).  VERIFY LGA-8 land pattern vs DPS368 DS Fig.18 before layout."
+    (at 120 175 0)
     (effects (font (size 1.27 1.27)) (justify left bottom))
   )
@@
 			)
 		)
-		(property "Value" "4.7k"
+		(property "Value" "2.2k"
 			(at 118.11 90.17 90)
 			(effects
@@
 			)
 		)
-		(property "LCSC" "C23162"
+		(property "LCSC" "C4190"
 			(at 118.11 90.17 0)
 			(hide yes)
@@
 			)
 		)
-		(property "MPN" "0603WAF4701T5E"
+		(property "MPN" "0603WAF2201T5E"
 			(at 118.11 90.17 0)
 			(hide yes)
@@
 			)
 		)
-		(property "Value" "4.7k"
+		(property "Value" "2.2k"
 			(at 110.49 90.17 90)
 			(effects
@@
 			)
 		)
-		(property "LCSC" "C23162"
+		(property "LCSC" "C4190"
 			(at 110.49 90.17 0)
 			(hide yes)
@@
 			)
 		)
-		(property "MPN" "0603WAF4701T5E"
+		(property "MPN" "0603WAF2201T5E"
 			(at 110.49 90.17 0)
 			(hide yes)
