File: hardware/kicad/stm32_core.kicad_sch (KiCad schematic)
At the start: 22 parts, among them J201 SWD, Q201 2N7002, U201 STM32F405RGT6, Y201 8MHz

Commit message: Review fixes: series protection R, I2C1 2.2k, C102 50V, gate & buck soft-start
7.f - PA2/PA3 = TTa (not 5V tolerant), PD2 = FT (5V tolerant) per STM32F405
DS8626. Add series R on the STM32 pin side: R205 1k ESC_TLM, R206 1k GPS_TX,
R207 1k GPS_RX (limits fault injection into PA2/PA3 to ~1.2 mA on a 5V UART).

3.a - Cross-domain series R: R208 470 BRIDGE_TX, R209 470 BRIDGE_RX, R210 470
ESP_STM_NRST (R203 pull-down + Q201 gate kept on the local node -> ESP-absent
fail-safe preserved).

6.a - I2C1 pull-ups R401/R402 4.7k -> 2.2k (C4190). With J703 cabled
(~90-100 pF): t_r ~= 186 ns < 300 ns (400 kHz); sink 1.4 mA at VOL.

1.a - C102 10uF 25V -> 50V (C138687), for 4S input transients + DC-bias
derating.

7.a - Inrush handled by a BUILD REQUIREMENT: anti-spark XT60/XT90 on the
battery lead (a single reverse-polarity P-FET cannot soft-start plug-in
inrush - body diode is forward). C114 100nF gate-source stays for a
controlled ~7 ms gate turn-on / softer VBAT_SW rise. J101 annotated.

MP2307 SS: C115 100nF on the SS pin (was left open). t_ss ~= 15 ms per r1.9
-> +5V ramps 0->5 V charging C105+C113 (~46 uF) at ~15 mA, not the ~4 A
current limit. Project symbol MP2307DN pin 8 corrected NC -> SS (passive).

ERC: 0 errors / 0 isolated_pin_label / 2 known pin_to_pin warnings.

Co-Authored-By: Claude Sonnet 5 <noreply@anthropic.com>
Claude-Session: https://claude.ai/code/session_0171uwNh8K8uwZuWio9f35u1
Parts:
- added R205, R206, R207: 1k, Resistor_SMD:R_0603_1608Metric, symbol Device:R
- added R208, R209, R210: 470, Resistor_SMD:R_0603_1608Metric, symbol Device:R
Connections:
- net BRIDGE_RX: now also R209.2; no longer U201.43 (PA10)
- net BRIDGE_TX: now also R208.2; no longer U201.42 (PA9)
- net ESC_TLM: now also R205.2; no longer U201.54 (PD2)
- net ESP_STM_NRST: now also R210.1; no longer Q201.1 (G), R203.1
- net GPS_RX: now also R207.2; no longer U201.17 (PA3)
- net GPS_TX: now also R206.2; no longer U201.16 (PA2)
- new net BRIDGE_RX_MCU: R209.1, U201.43 (PA10)
- new net BRIDGE_TX_MCU: R208.1, U201.42 (PA9)
- new net ESC_TLM_MCU: R205.1, U201.54 (PD2)
- new net ESP_STM_NRST_G: Q201.1 (G), R203.1, R210.2
- new net GPS_RX_MCU: R207.1, U201.17 (PA3)
- new net GPS_TX_MCU: R206.1, U201.16 (PA2)
Other:
- note added: "Series protection resistors (STM32-pin side): R205 1k ESC_TLM -> PD2 (PD2 is FT / 5 V tolerant; R is ESD + fault limit) R206 1k GPS_TX -> PA2 PA2/PA3 = TTa (ADC), NOT 5 V tolerant - R limits R207 1k GPS_RX -> PA3 fault injection to ~1.2 mA if a 5 V UART is plugged R208 470 BRIDGE_TX -> PA9 cross-domain (STM32 +3V3_SYS <-> ESP32 +3V3_ESP): R209 470 BRIDGE_RX -> PA10 limits current through the pin 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"
